File: kicad/ecg-instru/conditioning.kicad_sch (KiCad schematic)
At the start: 42 parts, among them J5 Conn_01x02_Socket, J6 Conn_01x02_Socket, J7 Conn_01x03_Socket, J8 Conn_01x03_Socket, U1 LM358, U2 LM358, U3 LM358, U5 INA114

Commit message: Board layout + Schematic + ESP32 initial src
Parts:
- removed J5, J6: Conn_01x02_Socket, Connector_PinHeader_2.54mm:PinHeader_1x02_P2.54mm_Vertical, symbol Connector:Conn_01x02_Socket
- added J4, J5: Conn_01x01_Socket, Connector_PinHeader_2.54mm:PinHeader_1x01_P2.54mm_Vertical, symbol Connector:Conn_01x01_Socket
- D1: footprint (none) -> Diode_THT:D_DO-41_SOD81_P10.16mm_Horizontal
- J7, J8: footprint (none) -> Connector_PinHeader_2.54mm:PinHeader_1x03_P2.54mm_Vertical
- R11, R12, R13, R14, R15, R16, R17, R18, R19, R20, R23, R24, R25, R27, R4, R5, R6, R7, R8, R9: footprint Resistor_THT:R_Axial_DIN0309_L9.0mm_D3.2mm_P15.24mm_Horizontal -> Resistor_THT:R_Axial_DIN0309_L9.0mm_D3.2mm_P12.70mm_Horizontal
- RV1, RV2, RV3, RV4: footprint Potentiometer_THT:Potentiometer_ACP_CA9-V10_Vertical -> Potentiometer_THT:Potentiometer_Bourns_3296W_Vertical
Connections:
- net COM: now also U2.2 (-); no longer U2.6 (-)
- net GNDREF: now also U2.3 (+), U2.6 (-), U2.7; no longer U2.1, U2.2 (-), U2.5 (+)
- net RL: now also U2.1; no longer U2.7
- net at C10.1, C11.1, R13.2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: now also J4.1 (Pin_1)
- net at R14.2, R15.1: now also U2.5 (+); no longer U2.3 (+)
- net U1A_VIN: no longer names the net of C12.2, R16.1, U1.5 (+)
- net U1A_VOUT: no longer names the net of R18.1, R19.1, U1.7, U3.3 (+)
- net U1A_VOUT: now also J5.1 (Pin_1)
- no-connect marks 3 -> 4
