File: kicad/ecg-instru/ecg-instru.kicad_pcb (KiCad board)
At the start: 2 copper layers, 100 x 100 mm, 46 parts, among them J1 Screw_Terminal_01x02, J2 Screw_Terminal_01x03, J3 Conn_01x04_Socket, J4 Screw_Terminal_01x02, J5 Conn_01x02_Socket, J6 Conn_01x02_Socket, U1 LM358, U2 LM358, U3 LM358, U5 INA114, U6 ESP32-DEVKIT-V1

Commit message: Board layout + Schematic + ESP32 initial src
Parts:
- removed C4: 100n, Capacitor_THT:C_Rect_L7.0mm_W2.5mm_P5.00mm
- removed R10: 220k, Resistor_THT:R_Axial_DIN0309_L9.0mm_D3.2mm_P15.24mm_Horizontal
- added C14: 100n, Capacitor_THT:C_Rect_L7.0mm_W2.5mm_P5.00mm, F.Cu at (133.1, 129.6)
- added D1: 3V3, Diode_THT:D_DO-41_SOD81_P10.16mm_Horizontal, F.Cu at (194.9, 98.4)
- added J7: Conn_01x03_Socket, Connector_PinHeader_2.54mm:PinHeader_1x03_P2.54mm_Vertical, F.Cu at (113.7, 94.7)
- added J8: Conn_01x03_Socket, Connector_PinHeader_2.54mm:PinHeader_1x03_P2.54mm_Vertical, F.Cu at (117.7, 94.7)
- added R23: 12k, Resistor_THT:R_Axial_DIN0309_L9.0mm_D3.2mm_P12.70mm_Horizontal, F.Cu at (108.7, 78.7)
- added R24: 12k, Resistor_THT:R_Axial_DIN0309_L9.0mm_D3.2mm_P12.70mm_Horizontal, F.Cu at (122.7, 91.4)
- added R25: 1k, Resistor_THT:R_Axial_DIN0309_L9.0mm_D3.2mm_P12.70mm_Horizontal, F.Cu at (163.4, 109.9)
- added R27: 1k, Resistor_THT:R_Axial_DIN0309_L9.0mm_D3.2mm_P12.70mm_Horizontal, F.Cu at (190.9, 109.9)
- added RV3: 1k, Potentiometer_THT:Potentiometer_Bourns_3296W_Vertical, F.Cu at (175.4, 120.9)
- added RV4: 2k, Potentiometer_THT:Potentiometer_Bourns_3296W_Vertical, F.Cu at (180.7, 130.4)
- C5, C6, C8, C9: value 12n -> 47n
- J3: value Conn_01x04_Socket -> Conn_01x02_Socket; footprint Connector_PinHeader_2.54mm:PinHeader_1x04_P2.54mm_Vertical -> Connector_PinHeader_2.54mm:PinHeader_1x02_P2.54mm_Vertical
- J4: value Screw_Terminal_01x02 -> Conn_01x01_Socket; footprint TerminalBlock:TerminalBlock_MaiXu_MX126-5.0-02P_1x02_P5.00mm -> Connector_PinHeader_2.54mm:PinHeader_1x01_P2.54mm_Vertical
- J5: value Conn_01x02_Socket -> Conn_01x01_Socket; footprint Connector_PinHeader_2.54mm:PinHeader_1x02_P2.54mm_Vertical -> Connector_PinHeader_2.54mm:PinHeader_1x01_P2.54mm_Vertical
- J6: value Conn_01x02_Socket -> Conn_01x06_Socket; footprint Connector_PinHeader_2.54mm:PinHeader_1x02_P2.54mm_Vertical -> Connector_PinHeader_2.54mm:PinHeader_1x06_P2.54mm_Vertical
- R1, R14, R15, R16, R18, R2, R20, R3, R7, R9: footprint Resistor_THT:R_Axial_DIN0309_L9.0mm_D3.2mm_P15.24mm_Horizontal -> Resistor_THT:R_Axial_DIN0309_L9.0mm_D3.2mm_P12.70mm_Horizontal
- R11, R13, R17, R19: value 1k -> 10k; footprint Resistor_THT:R_Axial_DIN0309_L9.0mm_D3.2mm_P15.24mm_Horizontal -> Resistor_THT:R_Axial_DIN0309_L9.0mm_D3.2mm_P12.70mm_Horizontal
- R12, R6: value 220k -> 56k; footprint Resistor_THT:R_Axial_DIN0309_L9.0mm_D3.2mm_P15.24mm_Horizontal -> Resistor_THT:R_Axial_DIN0309_L9.0mm_D3.2mm_P12.70mm_Horizontal
- R4, R5: value 100 -> 1k; footprint Resistor_THT:R_Axial_DIN0309_L9.0mm_D3.2mm_P15.24mm_Horizontal -> Resistor_THT:R_Axial_DIN0309_L9.0mm_D3.2mm_P12.70mm_Horizontal
- R8: value 220k -> 27k; footprint Resistor_THT:R_Axial_DIN0309_L9.0mm_D3.2mm_P15.24mm_Horizontal -> Resistor_THT:R_Axial_DIN0309_L9.0mm_D3.2mm_P12.70mm_Horizontal
- RV1, RV2: footprint Potentiometer_THT:Potentiometer_ACP_CA9-V10_Vertical -> Potentiometer_THT:Potentiometer_Bourns_3296W_Vertical
- moved J6 266.7 mm to (141.4, 55.0), turned to 90 degrees
- moved R5 254.4 mm to (117.8, 91.4), turned to 90 degrees
- moved R4 248.3 mm to (113.6, 78.7), turned to -90 degrees
- moved R19 243.4 mm to (158.9, 119.4), turned to -90 degrees
- moved R18 236.1 mm to (154.0, 120.0), turned to 180 degrees
- moved U5 231.6 mm to (111.4, 99.9)
- moved R16 221.4 mm to (150.3, 128.8), turned to -90 degrees
- moved R17 219.7 mm to (154.4, 141.5), turned to 90 degrees
- moved J5 206.8 mm to (143.6, 135.9), turned to 180 degrees
- moved C2 202.0 mm to (140.8, 96.1)
- moved RV2 191.8 mm to (171.0, 101.0), turned to 90 degrees
- moved R13 189.2 mm to (116.5, 124.8)
- moved C12 184.0 mm to (141.3, 125.1)
- moved R7 181.9 mm to (123.4, 115.6), turned to 180 degrees
- moved R12 181.4 mm to (191.0, 119.3), turned to -90 degrees
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Connections:
- net Net-(J2-Pin_2) renamed RA_E
- C1 pad 2: Net-(J2-Pin_1) -> RL_E
- C10 pad 1: Net-(J5-Pin_2) -> Net-(J4-Pin_1)
- C11 pad 1: Net-(J5-Pin_2) -> Net-(J4-Pin_1)
- C12 pad 2: /Conditioning/U1A_VIN -> Net-(U1B-+)
- C6 pad 2: Net-(U3B--) -> GNDREF
- C7 pad 2: Net-(J5-Pin_1) -> Net-(U1A-+)
- C8 pad 2: Net-(U3B--) -> GNDREF
- C9 pad 1: Net-(U3A-+) -> Net-(U3B-+)
- J2 pad 1: Net-(J2-Pin_1) -> LA_E
- J2 pad 3: Net-(J2-Pin_3) -> RL_E
- J3 pad 1: I2C1_SCL -> VADC
- J3 pad 2: I2C1_SDA -> VSENSE
- J4 pad 1: B0 -> Net-(J4-Pin_1)
- J6 pad 1: /Conditioning/U1A_VIN -> B1
- J6 pad 2: VSENSE -> B0
- R1 pad 1: Net-(J2-Pin_3) -> LA_E
- R1 pad 2: RA -> LA
- R12 pad 2: Net-(U3A-+) -> Net-(U3B-+)
- R13 pad 2: Net-(J5-Pin_2) -> Net-(J4-Pin_1)
- R14 pad 2: Net-(U2A-+) -> Net-(U2B-+)
- R15 pad 1: Net-(U2A-+) -> Net-(U2B-+)
- R16 pad 1: /Conditioning/U1A_VIN -> Net-(U1B-+)
- R18 pad 1: VSENSE -> Net-(J5-Pin_1)
- R19 pad 1: VSENSE -> Net-(J5-Pin_1)
- R2 pad 2: LA -> RA
- R3 pad 1: Net-(J2-Pin_1) -> RL_E
- R4 pad 2: Net-(R4-Pad2) -> Net-(J7-Pin_1)
- R5 pad 1: COM -> Net-(J8-Pin_1)
- R5 pad 2: Net-(R5-Pad2) -> COM
- R6 pad 2: Net-(C6-Pad1) -> Net-(R6-Pad2)
- R8 pad 2: Net-(U3B--) -> Net-(R8-Pad2)
- R9 pad 2: Net-(J5-Pin_1) -> Net-(U1A-+)
- RV2 pad 1: GNDREF -> VSENSE
- RV2 pad 2: Net-(U3B-+) -> Net-(U3A--)
- RV2 pad 3: VFILTER -> unconnected-(RV2-Pad3)
- U1 pad 1: Net-(J5-Pin_2) -> Net-(J4-Pin_1)
- U1 pad 3: Net-(J5-Pin_1) -> Net-(U1A-+)
- U1 pad 5: /Conditioning/U1A_VIN -> Net-(U1B-+)
- U1 pad 7: VSENSE -> Net-(J5-Pin_1)
- U2 pad 1: GNDREF -> RL
- U2 pad 2: GNDREF -> COM
- U2 pad 3: Net-(U2A-+) -> GNDREF
- U2 pad 5: 0 -> Net-(U2B-+)
- U2 pad 6: COM -> GNDREF
- U2 pad 7: RL -> GNDREF
- U3 pad 1: VFILTER -> VSENSE
- U3 pad 2: VFILTER -> Net-(U3A--)
- U3 pad 3: Net-(U3A-+) -> Net-(J5-Pin_1)
- U5 pad 1: Net-(R4-Pad2) -> Net-(J7-Pin_2)
- U5 pad 8: Net-(R5-Pad2) -> Net-(J8-Pin_2)
- U6 pad 10: I2C1_SCL -> unconnected-(U6-D19-Pad10)
- U6 pad 11: I2C1_SDA -> unconnected-(U6-D21-Pad11)
- U6 pad 12: unconnected-(U6-RX0-Pad12) -> I2C1_SDA
- U6 pad 13: unconnected-(U6-TX0-Pad13) -> I2C1_SCL
- U6 pad 14: unconnected-(U6-D22-Pad14) -> B0
- U6 pad 15: unconnected-(U6-D23-Pad15) -> B1
- U6 pad 20: VFILTER -> VADC
Routing:
- net +5V: track 0.00 -> 369.9 mm, vias 0 -> 2
- net GNDREF: track 0.00 -> 255.7 mm
- net VSENSE: track 0.00 -> 94.1 mm
- net COM: track 0.00 -> 62.4 mm
- net Net-(J5-Pin_1): track 0.00 -> 58.3 mm
- net RL: track 0.00 -> 51.7 mm
- net VADC: track 0.00 -> 51.4 mm
- net RA: track 0.00 -> 47.6 mm
- net Net-(U3B-+): track 0.00 -> 38.6 mm
- net Net-(U1B--): track 0.00 -> 36.9 mm
- net LA: track 0.00 -> 35.7 mm
- net 0: track 0.00 -> 32.0 mm, vias 0 -> 7
- net Net-(U1A-+): track 0.00 -> 24.4 mm
- net Net-(U1B-+): track 0.00 -> 24.1 mm
- net Net-(J4-Pin_1): track 0.00 -> 22.0 mm
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- added copper zone on B.Cu, net 0
Other:
- board text added: "Front-End - Heartbeat monitor V1 UFRGS - DELET - 2025/1 Fernando Welzel Guilherme Huth Tales Ramos"
